File: MotorController.kicad_sch (KiCad schematic)
At the start: 133 parts, among them IC1 ft234xd, IC2 A3921KLPTR-T, IC3 A3921KLPTR-T, J1 SH, J10 PA, J11 XT30, J2 USB_B_Micro, J3 XA, J4 XA, J5 3020-10-0300-00, J6 SH, J7 SH, J8 3020-10-0300-00, J9 XA, Q1 GSFQ6806, Q2 GSFQ6806, Q3 GSFQ6806, Q4 SFS9Z34, Q5 GSFQ6806, Q6 SFS9Z34, SW2 BLACK, SW3 BLACK, SW4 2MS1-T1-B4-VS2-Q-E-S, SW5 RED, U1 LXES11D, U2 STM32F303K8Tx, U3 TJA1441AT, U4 TPSM13604HNDWR, U5 LMZ12002EXT, Y1 32M

Commit message: GND 以外の配線をとりあえずやった。水晶の下の配線をなくした。パーツ同士の干渉をなくした。
Parts:
- removed R8: R, Resistor_SMD:R_0603_1608Metric, symbol Device:R
Changed lines of the file:
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@@
-    )
-  )
-  (symbol (lib_id "Device:R") (at 21.59 71.12 0) (unit 1)
-    (in_bom yes) (on_board yes) (dnp no) (fields_autoplaced)
-    (property "Reference" "R8" (at 24.13 69.85 0)
-      (effects (font (size 1.27 1.27)) (justify left))
-    )
-    (property "Value" "R" (at 24.13 72.39 0)
-      (effects (font (size 1.27 1.27)) (justify left))
-    )
-    (property "Footprint" "Resistor_SMD:R_0603_1608Metric" (at 19.812 71.12 90)
-      (effects (font (size 1.27 1.27)) hide)
-    )
-    (property "Datasheet" "~" (at 21.59 71.12 0)
-      (effects (font (size 1.27 1.27)) hide)
-    )
-    (pin "1")
-    (pin "2")
-    (instances
-      (project "MotorController"
-        (path "/5f98a318-5528-4c4b-bcf3-90ead89a063c"
-          (reference "R8") (unit 1)
-        )
-      )
     )
   )
